File: circuits/TrainingTracer/power.kicad_sch (KiCad schematic)
At the start: 13 parts, among them J1 Conn_01x02, SW1 SW_SPDT, U1 NJU7223F-33, U2 LM2931-3.3_TO220

Commit message: 回路完成
Parts:
- removed J1: Conn_01x02, symbol Connector_Generic:Conn_01x02
- added J1: BATT+, Connector_Wire:SolderWire-0.75sqmm_1x01_D1.25mm_OD2.3mm, symbol Connector_Generic:Conn_01x01
- added J10, J3, J4, J5, J6, J7, J8, J9: Conn_01x01_Socket, Connector_Wire:SolderWire-0.25sqmm_1x01_D0.65mm_OD1.7mm, symbol Connector:Conn_01x01_Socket
- added J2: BATT-, Connector_Wire:SolderWire-0.75sqmm_1x01_D1.25mm_OD2.3mm, symbol Connector_Generic:Conn_01x01
- added R18: 0, TrainingTracer:jmp_15.24mm, symbol Device:R_US
- C1: footprint (none) -> Capacitor_THT:CP_Radial_D6.3mm_P2.50mm
- C2: value C_Small -> 0.33uF; footprint (none) -> Capacitor_THT:C_Disc_D5.0mm_W2.5mm_P5.00mm
- C3, C4: value C_Small -> 0.1uF; footprint (none) -> Capacitor_THT:C_Disc_D5.0mm_W2.5mm_P5.00mm
- D1: value LED_Filled -> LED_BLUE; footprint (none) -> LED_THT:LED_D3.0mm
- D2: footprint (none) -> Diode_THT:D_A-405_P7.62mm_Horizontal
- R1: value R_Small_US -> 1k; footprint (none) -> Resistor_THT:R_Axial_DIN0207_L6.3mm_D2.5mm_P10.16mm_Horizontal
- R2: value R_Small_US -> 20k; footprint (none) -> Resistor_THT:R_Axial_DIN0204_L3.6mm_D1.6mm_P7.62mm_Horizontal
- R3: value R_Small_US -> 10k; footprint (none) -> Resistor_THT:R_Axial_DIN0204_L3.6mm_D1.6mm_P7.62mm_Horizontal
- SW1: footprint (none) -> TrainingTracer:Switch
- U1: footprint (none) -> Package_TO_SOT_THT:TO-220-3_Vertical
Connections:
- net +3.3V: now also J3.1 (Pin_1), J4.1 (Pin_1)
- net +BATT: now also J1.1 (Pin_1), R18.1; no longer SW1.2 (B)
- net GND: now also J10.1 (Pin_1), J2.1 (Pin_1), J7.1 (Pin_1), J8.1 (Pin_1), J9.1 (Pin_1)
- net VCC: now also J5.1 (Pin_1), J6.1 (Pin_1)
- new net: R18.2, SW1.2 (B)

Commit message: PCBのPDF出力
Other:
- note added: "一般的なピン配置のレギュレータ"
- note added: "改良箇所1：パイロットランプ"
- note added: "改良箇所2：バッテリー電圧計測値のズレ対策"
- note added: "改造箇所1：汎用レギュレータ(M78AR033-0.5等)への対応"
- note added: "改造箇所2：改造・テスト用ピンアウト"
- note added: "逆電圧防止Di(SBD推奨)"
- moved on the sheet: J10, J3, J4, J5, J6, J7, J8, J9, U2
